Commit message: it seams to work

File: franka_selfcollision/urdfs/fr3_duo.urdf (robot description, URDF)
Before this commit: robot fr3_duo, 31 links, 30 joints
Links:
- removed link cover_link
- added link left_fr3v2_link0_accelerometer_bottom
- added link left_fr3v2_link0_accelerometer_top
- added link left_fr3v2_link1_accelerometer_bottom
- added link left_fr3v2_link1_accelerometer_top
- added link left_fr3v2_link2_accelerometer_bottom
- added link left_fr3v2_link2_accelerometer_top
- added link left_fr3v2_link3_accelerometer_bottom
- added link left_fr3v2_link3_accelerometer_top
- added link left_fr3v2_link4_accelerometer_bottom
- added link left_fr3v2_link4_accelerometer_top
- added link left_fr3v2_link5_accelerometer_bottom
- added link left_fr3v2_link5_accelerometer_top
- added link right_fr3v2_link0_accelerometer_bottom
- added link right_fr3v2_link0_accelerometer_top
- added link right_fr3v2_link1_accelerometer_bottom
- added link right_fr3v2_link1_accelerometer_top
- added link right_fr3v2_link2_accelerometer_bottom
- added link right_fr3v2_link2_accelerometer_top
- added link right_fr3v2_link3_accelerometer_bottom
- added link right_fr3v2_link3_accelerometer_top
- added link right_fr3v2_link4_accelerometer_bottom
- added link right_fr3v2_link4_accelerometer_top
- added link right_fr3v2_link5_accelerometer_bottom
- added link right_fr3v2_link5_accelerometer_top
- link mount_link: mass 4.972778 -> 4.093846; geometry collision mesh filename=package://franka_description/meshes/accessories/fr3_duo_mou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; collision mesh filename=package://franka_description/meshes/accessories/fr3_duo_mou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
Joints:
- removed joint cover_joint
- added joint left_fr3v2_link0_accelerometer_bottom_joint: type fixed, parent left_fr3v2_link0, child left_fr3v2_link0_accelerometer_bottom, origin xyz=0 0 0.06 rpy=0 0 0
- added joint left_fr3v2_link0_accelerometer_top_joint: type fixed, parent left_fr3v2_link0, child left_fr3v2_link0_accelerometer_top, origin xyz=0 0 0.05 rpy=3.14159 0 0
- added joint left_fr3v2_link1_accelerometer_bottom_joint: type fixed, parent left_fr3v2_link1, child left_fr3v2_link1_accelerometer_bottom, origin xyz=0 -0.09 0.0 rpy=-1.5708 0 0
- added joint left_fr3v2_link1_accelerometer_top_joint: type fixed, parent left_fr3v2_link1, child left_fr3v2_link1_accelerometer_top, origin xyz=0 -0.1 0.0 rpy=1.5708 0 0
- added joint left_fr3v2_link2_accelerometer_bottom_joint: type fixed, parent left_fr3v2_link2, child left_fr3v2_link2_accelerometer_bottom, origin xyz=0 -0.14 0 rpy=1.5708 0 0
- added joint left_fr3v2_link2_accelerometer_top_joint: type fixed, parent left_fr3v2_link2, child left_fr3v2_link2_accelerometer_top, origin xyz=0 -0.13 0 rpy=-1.5708 0 0
- added joint left_fr3v2_link3_accelerometer_bottom_joint: type fixed, parent left_fr3v2_link3, child left_fr3v2_link3_accelerometer_bottom, origin xyz=0.0825 0.04 0 rpy=1.5708 0 0
- added joint left_fr3v2_link3_accelerometer_top_joint: type fixed, parent left_fr3v2_link3, child left_fr3v2_link3_accelerometer_top, origin xyz=0.0825 0.05 0 rpy=-1.5708 0 0
- added joint left_fr3v2_link4_accelerometer_bottom_joint: type fixed, parent left_fr3v2_link4, child left_fr3v2_link4_accelerometer_bottom, origin xyz=-0.0825 0.06 0 rpy=-1.5708 0 0
- added joint left_fr3v2_link4_accelerometer_top_joint: type fixed, parent left_fr3v2_link4, child left_fr3v2_link4_accelerometer_top, origin xyz=-0.0825 0.05 0 rpy=1.5708 0 0
- added joint left_fr3v2_link5_accelerometer_bottom_joint: type fixed, parent left_fr3v2_link5, child left_fr3v2_link5_accelerometer_bottom, origin xyz=0 0.1 0 rpy=1.5708 0 0
- added joint left_fr3v2_link5_accelerometer_top_joint: type fixed, parent left_fr3v2_link5, child left_fr3v2_link5_accelerometer_top, origin xyz=0 0.11 0 rpy=-1.5708 0 0
- added joint right_fr3v2_link0_accelerometer_bottom_joint: type fixed, parent right_fr3v2_link0, child right_fr3v2_link0_accelerometer_bottom, origin xyz=0 0 0.06 rpy=0 0 0
- added joint right_fr3v2_link0_accelerometer_top_joint: type fixed, parent right_fr3v2_link0, child right_fr3v2_link0_accelerometer_top, origin xyz=0 0 0.05 rpy=3.14159 0 0
- added joint right_fr3v2_link1_accelerometer_bottom_joint: type fixed, parent right_fr3v2_link1, child right_fr3v2_link1_accelerometer_bottom, origin xyz=0 -0.09 0.0 rpy=-1.5708 0 0
- added joint right_fr3v2_link1_accelerometer_top_joint: type fixed, parent right_fr3v2_link1, child right_fr3v2_link1_accelerometer_top, origin xyz=0 -0.1 0.0 rpy=1.5708 0 0
- added joint right_fr3v2_link2_accelerometer_bottom_joint: type fixed, parent right_fr3v2_link2, child right_fr3v2_link2_accelerometer_bottom, origin xyz=0 -0.14 0 rpy=1.5708 0 0
- added joint right_fr3v2_link2_accelerometer_top_joint: type fixed, parent right_fr3v2_link2, child right_fr3v2_link2_accelerometer_top, origin xyz=0 -0.13 0 rpy=-1.5708 0 0
- added joint right_fr3v2_link3_accelerometer_bottom_joint: type fixed, parent right_fr3v2_link3, child right_fr3v2_link3_accelerometer_bottom, origin xyz=0.0825 0.04 0 rpy=1.5708 0 0
- added joint right_fr3v2_link3_accelerometer_top_joint: type fixed, parent right_fr3v2_link3, child right_fr3v2_link3_accelerometer_top, origin xyz=0.0825 0.05 0 rpy=-1.5708 0 0
- added joint right_fr3v2_link4_accelerometer_bottom_joint: type fixed, parent right_fr3v2_link4, child right_fr3v2_link4_accelerometer_bottom, origin xyz=-0.0825 0.06 0 rpy=-1.5708 0 0
- added joint right_fr3v2_link4_accelerometer_top_joint: type fixed, parent right_fr3v2_link4, child right_fr3v2_link4_accelerometer_top, origin xyz=-0.0825 0.05 0 rpy=1.5708 0 0
- added joint right_fr3v2_link5_accelerometer_bottom_joint: type fixed, parent right_fr3v2_link5, child right_fr3v2_link5_accelerometer_bottom, origin xyz=0 0.1 0 rpy=1.5708 0 0
- added joint right_fr3v2_link5_accelerometer_top_joint: type fixed, parent right_fr3v2_link5, child right_fr3v2_link5_accelerometer_top, origin xyz=0 0.11 0 rpy=-1.5708 0 0
- joint left_base_joint: origin xyz=0.03467 0.050681 0.202 rpy=-0.89334809 -0.17456074 -0.46334506 -> xyz=0.0369 0.05018 0.050885 rpy=-0.89334809 -0.17456074 -0.46334506
- joint right_base_joint: origin xyz=0.03467 -0.050681 0.202 rpy=0.89334809 -0.17456074 0.46334506 -> xyz=0.0369 -0.05018 0.050885 rpy=0.89334809 -0.17456074 0.46334506
