Commit message: self collision now with xacro files

File: franka_selfcollision/urdfs/fr3_duo.urdf (robot description, URDF)
Before this commit: robot fr3_duo, 54 links, 53 joints
Links:
- removed link left_fr3v2_hand
- removed link left_fr3v2_hand_tcp
- removed link left_fr3v2_leftfinger
- removed link left_fr3v2_link0
- removed link left_fr3v2_link0_accelerometer_bottom
- removed link left_fr3v2_link0_accelerometer_top
- removed link left_fr3v2_link1
- removed link left_fr3v2_link1_accelerometer_bottom
- removed link left_fr3v2_link1_accelerometer_top
- removed link left_fr3v2_link2
- removed link left_fr3v2_link2_accelerometer_bottom
- removed link left_fr3v2_link2_accelerometer_top
- removed link left_fr3v2_link3
- removed link left_fr3v2_link3_accelerometer_bottom
- removed link left_fr3v2_link3_accelerometer_top
- removed link left_fr3v2_link4
- removed link left_fr3v2_link4_accelerometer_bottom
- removed link left_fr3v2_link4_accelerometer_top
- removed link left_fr3v2_link5
- removed link left_fr3v2_link5_accelerometer_bottom
- removed link left_fr3v2_link5_accelerometer_top
- removed link left_fr3v2_link6
- removed link left_fr3v2_link7
- removed link left_fr3v2_link8
- removed link left_fr3v2_rightfinger
- removed link right_fr3v2_hand
- removed link right_fr3v2_hand_tcp
- removed link right_fr3v2_leftfinger
- removed link right_fr3v2_link0
- removed link right_fr3v2_link0_accelerometer_bottom
- removed link right_fr3v2_link0_accelerometer_top
- removed link right_fr3v2_link1
- removed link right_fr3v2_link1_accelerometer_bottom
- removed link right_fr3v2_link1_accelerometer_top
- removed link right_fr3v2_link2
- removed link right_fr3v2_link2_accelerometer_bottom
- removed link right_fr3v2_link2_accelerometer_top
- removed link right_fr3v2_link3
- removed link right_fr3v2_link3_accelerometer_bottom
- removed link right_fr3v2_link3_accelerometer_top
- removed link right_fr3v2_link4
- removed link right_fr3v2_link4_accelerometer_bottom
- removed link right_fr3v2_link4_accelerometer_top
- removed link right_fr3v2_link5
- removed link right_fr3v2_link5_accelerometer_bottom
- removed link right_fr3v2_link5_accelerometer_top
- removed link right_fr3v2_link6
- removed link right_fr3v2_link7
- removed link right_fr3v2_link8
- removed link right_fr3v2_rightfinger
- added link left_fr3_hand, mass 0.6544; collision mesh filename=package://franka_description/meshes/robot_ee/franka_hand_wh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; visual mesh filename=package://franka_description/meshes/robot_ee/franka_hand_wh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
- added link left_fr3_hand_tcp
- added link left_fr3_leftfinger, mass 0.0291; collision box size=17.5e-3 15.2e-3 18.5e-3; collision box size=17.5e-3 7e-3 23.5e-3
- added link left_fr3_link0, mass 2.3966; collision mesh filename=package://franka_description/meshes/robot_arms/fr3/collisio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; visual mesh filename=package://franka_description/meshes/robot_arms/fr3/visual/l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
- added link left_fr3_link0_accelerometer_bottom
- added link left_fr3_link0_accelerometer_top
- added link left_fr3_link1, mass 2.4377; collision mesh filename=package://franka_description/meshes/robot_arms/fr3/collisio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; visual mesh filename=package://franka_description/meshes/robot_arms/fr3/visual/l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
- added link left_fr3_link1_accelerometer_bottom
- added link left_fr3_link1_accelerometer_top
- added link left_fr3_link2, mass 2.2375; collision mesh filename=package://franka_description/meshes/robot_arms/fr3/collisio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; visual mesh filename=package://franka_description/meshes/robot_arms/fr3/visual/l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
- added link left_fr3_link2_accelerometer_bottom
- added link left_fr3_link2_accelerometer_top
- added link left_fr3_link3, mass 2.193082; collision mesh filename=package://franka_description/meshes/robot_arms/fr3/collisio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; visual mesh filename=package://franka_description/meshes/robot_arms/fr3/visual/l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
- added link left_fr3_link3_accelerometer_bottom
- added link left_fr3_link3_accelerometer_top
- added link left_fr3_link4, mass 2.181537; collision mesh filename=package://franka_description/meshes/robot_arms/fr3/collisio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; visual mesh filename=package://franka_description/meshes/robot_arms/fr3/visual/l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
- added link left_fr3_link4_accelerometer_bottom
- added link left_fr3_link4_accelerometer_top
- added link left_fr3_link5, mass 2.186881; collision mesh filename=package://franka_description/meshes/robot_arms/fr3/collisio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; visual mesh filename=package://franka_description/meshes/robot_arms/fr3/visual/l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
- added link left_fr3_link5_accelerometer_bottom
- added link left_fr3_link5_accelerometer_top
- added link left_fr3_link6, mass 1.579681; collision mesh filename=package://franka_description/meshes/robot_arms/fr3/collisio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; visual mesh filename=package://franka_description/meshes/robot_arms/fr3/visual/l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
- added link left_fr3_link7, mass 0.694841; collision mesh filename=package://franka_description/meshes/robot_arms/fr3/collisio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; visual mesh filename=package://franka_description/meshes/robot_arms/fr3/visual/l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
- added link left_fr3_link8
- added link left_fr3_rightfinger, mass 0.0291; collision box size=17.5e-3 15.2e-3 18.5e-3; collision box size=17.5e-3 7e-3 23.5e-3
- added link right_fr3_hand, mass 0.6544; collision mesh filename=package://franka_description/meshes/robot_ee/franka_hand_wh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; visual mesh filename=package://franka_description/meshes/robot_ee/franka_hand_wh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
- added link right_fr3_hand_tcp
- added link right_fr3_leftfinger, mass 0.0291; collision box size=17.5e-3 15.2e-3 18.5e-3; collision box size=17.5e-3 7e-3 23.5e-3
- added link right_fr3_link0, mass 2.3966; collision mesh filename=package://franka_description/meshes/robot_arms/fr3/collisio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; visual mesh filename=package://franka_description/meshes/robot_arms/fr3/visual/l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
- added link right_fr3_link0_accelerometer_bottom
- added link right_fr3_link0_accelerometer_top
- added link right_fr3_link1, mass 2.4377; collision mesh filename=package://franka_description/meshes/robot_arms/fr3/collisio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; visual mesh filename=package://franka_description/meshes/robot_arms/fr3/visual/l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
- added link right_fr3_link1_accelerometer_bottom
- added link right_fr3_link1_accelerometer_top
- added link right_fr3_link2, mass 2.2375; collision mesh filename=package://franka_description/meshes/robot_arms/fr3/collisio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; visual mesh filename=package://franka_description/meshes/robot_arms/fr3/visual/l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
- added link right_fr3_link2_accelerometer_bottom
- added link right_fr3_link2_accelerometer_top
- added link right_fr3_link3, mass 2.193082; collision mesh filename=package://franka_description/meshes/robot_arms/fr3/collisio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; visual mesh filename=package://franka_description/meshes/robot_arms/fr3/visual/l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
- added link right_fr3_link3_accelerometer_bottom
- added link right_fr3_link3_accelerometer_top
- added link right_fr3_link4, mass 2.181537; collision mesh filename=package://franka_description/meshes/robot_arms/fr3/collisio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; visual mesh filename=package://franka_description/meshes/robot_arms/fr3/visual/l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
- added link right_fr3_link4_accelerometer_bottom
- added link right_fr3_link4_accelerometer_top
- added link right_fr3_link5, mass 2.186881; collision mesh filename=package://franka_description/meshes/robot_arms/fr3/collisio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; visual mesh filename=package://franka_description/meshes/robot_arms/fr3/visual/l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
- added link right_fr3_link5_accelerometer_bottom
- added link right_fr3_link5_accelerometer_top
- added link right_fr3_link6, mass 1.579681; collision mesh filename=package://franka_description/meshes/robot_arms/fr3/collisio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; visual mesh filename=package://franka_description/meshes/robot_arms/fr3/visual/l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
- added link right_fr3_link7, mass 0.694841; collision mesh filename=package://franka_description/meshes/robot_arms/fr3/collisio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; visual mesh filename=package://franka_description/meshes/robot_arms/fr3/visual/l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
- added link right_fr3_link8
- added link right_fr3_rightfinger, mass 0.0291; collision box size=17.5e-3 15.2e-3 18.5e-3; collision box size=17.5e-3 7e-3 23.5e-3
Joints:
- removed joint left_fr3v2_finger_joint1
- removed joint left_fr3v2_finger_joint2
- removed joint left_fr3v2_hand_joint
- removed joint left_fr3v2_hand_tcp_joint
- removed joint left_fr3v2_joint1
- removed joint left_fr3v2_joint2
- removed joint left_fr3v2_joint3
- removed joint left_fr3v2_joint4
- removed joint left_fr3v2_joint5
- removed joint left_fr3v2_joint6
- removed joint left_fr3v2_joint7
- removed joint left_fr3v2_joint8
- removed joint left_fr3v2_left_base_joint
- removed joint left_fr3v2_link0_accelerometer_bottom_joint
- removed joint left_fr3v2_link0_accelerometer_top_joint
- removed joint left_fr3v2_link1_accelerometer_bottom_joint
- removed joint left_fr3v2_link1_accelerometer_top_joint
- removed joint left_fr3v2_link2_accelerometer_bottom_joint
- removed joint left_fr3v2_link2_accelerometer_top_joint
- removed joint left_fr3v2_link3_accelerometer_bottom_joint
- removed joint left_fr3v2_link3_accelerometer_top_joint
- removed joint left_fr3v2_link4_accelerometer_bottom_joint
- removed joint left_fr3v2_link4_accelerometer_top_joint
- removed joint left_fr3v2_link5_accelerometer_bottom_joint
- removed joint left_fr3v2_link5_accelerometer_top_joint
- removed joint right_fr3v2_finger_joint1
- removed joint right_fr3v2_finger_joint2
- removed joint right_fr3v2_hand_joint
- removed joint right_fr3v2_hand_tcp_joint
- removed joint right_fr3v2_joint1
- removed joint right_fr3v2_joint2
- removed joint right_fr3v2_joint3
- removed joint right_fr3v2_joint4
- removed joint right_fr3v2_joint5
- removed joint right_fr3v2_joint6
- removed joint right_fr3v2_joint7
- removed joint right_fr3v2_joint8
- removed joint right_fr3v2_link0_accelerometer_bottom_joint
- removed joint right_fr3v2_link0_accelerometer_top_joint
- removed joint right_fr3v2_link1_accelerometer_bottom_joint
- removed joint right_fr3v2_link1_accelerometer_top_joint
- removed joint right_fr3v2_link2_accelerometer_bottom_joint
- removed joint right_fr3v2_link2_accelerometer_top_joint
- removed joint right_fr3v2_link3_accelerometer_bottom_joint
- removed joint right_fr3v2_link3_accelerometer_top_joint
- removed joint right_fr3v2_link4_accelerometer_bottom_joint
- removed joint right_fr3v2_link4_accelerometer_top_joint
- removed joint right_fr3v2_link5_accelerometer_bottom_joint
- removed joint right_fr3v2_link5_accelerometer_top_joint
- removed joint right_fr3v2_right_base_joint
- added joint left_fr3_finger_joint1: type prismatic, parent left_fr3_hand, child left_fr3_leftfinger, origin xyz=0 0 0.0584 rpy=0 0 0, axis 0 1 0, limit lower=0.0 upper=0.04 effort=100 velocity=0.2
- added joint left_fr3_finger_joint2: type prismatic, parent left_fr3_hand, child left_fr3_rightfinger, origin xyz=0 0 0.0584 rpy=0 0 3.141592653589793, axis 0 1 0, limit lower=0.0 upper=0.04 effort=100 velocity=0.2, mimic joint=left_fr3_finger_joint1
- added joint left_fr3_hand_joint: type fixed, parent left_fr3_link8, child left_fr3_hand, origin xyz=0 0 0 rpy=0 0 -0.7853981633974483
- added joint left_fr3_hand_tcp_joint: type fixed, parent left_fr3_hand, child left_fr3_hand_tcp, origin xyz=0 0 0.1034 rpy=0 0 0
- added joint left_fr3_joint1: type revolute, parent left_fr3_link0, child left_fr3_link1, origin xyz=0 0 0.333 rpy=0 0 0, axis 0 0 1, limit lower=-2.9007400166666666 upper=2.9007400166666666 effort=87.0 velocity=2.62
- added joint left_fr3_joint2: type revolute, parent left_fr3_link1, child left_fr3_link2, origin xyz=0 0 0 rpy=-1.570796326794897 0 0, axis 0 0 1, limit lower=-1.8360900166666667 upper=1.8360900166666667 effort=87.0 velocity=2.62
- added joint left_fr3_joint3: type revolute, parent left_fr3_link2, child left_fr3_link3, origin xyz=0 -0.316 0 rpy=1.570796326794897 0 0, axis 0 0 1, limit lower=-2.9007400166666666 upper=2.9007400166666666 effort=87.0 velocity=2.62
- added joint left_fr3_joint4: type revolute, parent left_fr3_link3, child left_fr3_link4, origin xyz=0.0825 0 0 rpy=1.570796326794897 0 0, axis 0 0 1, limit lower=-3.077020016666667 upper=-0.11693708333333333 effort=87.0 velocity=2.62
- added joint left_fr3_joint5: type revolute, parent left_fr3_link4, child left_fr3_link5, origin xyz=-0.0825 0.384 0 rpy=-1.570796326794897 0 0, axis 0 0 1, limit lower=-2.87630335 upper=2.87630335 effort=12.0 velocity=5.26
- added joint left_fr3_joint6: type revolute, parent left_fr3_link5, child left_fr3_link6, origin xyz=0 0 0 rpy=1.570796326794897 0 0, axis 0 0 1, limit lower=0.43982265 upper=4.62163335 effort=12.0 velocity=4.18
- added joint left_fr3_joint7: type revolute, parent left_fr3_link6, child left_fr3_link7, origin xyz=0.088 0 0 rpy=1.570796326794897 0 0, axis 0 0 1, limit lower=-3.05083335 upper=3.05083335 effort=12.0 velocity=5.26
- added joint left_fr3_joint8: type fixed, parent left_fr3_link7, child left_fr3_link8, origin xyz=0 0 0.107 rpy=0 0 0
- added joint left_fr3_left_base_joint: type fixed, parent left_base, child left_fr3_link0, origin xyz=0 0 0 rpy=0 0 0
- added joint left_fr3_link0_accelerometer_bottom_joint: type fixed, parent left_fr3_link0, child left_fr3_link0_accelerometer_bottom, origin xyz=0 0 0.06 rpy=0 0 0
- added joint left_fr3_link0_accelerometer_top_joint: type fixed, parent left_fr3_link0, child left_fr3_link0_accelerometer_top, origin xyz=0 0 0.05 rpy=3.14159 0 0
- added joint left_fr3_link1_accelerometer_bottom_joint: type fixed, parent left_fr3_link1, child left_fr3_link1_accelerometer_bottom, origin xyz=0 -0.09 0.0 rpy=-1.5708 0 0
- added joint left_fr3_link1_accelerometer_top_joint: type fixed, parent left_fr3_link1, child left_fr3_link1_accelerometer_top, origin xyz=0 -0.1 0.0 rpy=1.5708 0 0
- added joint left_fr3_link2_accelerometer_bottom_joint: type fixed, parent left_fr3_link2, child left_fr3_link2_accelerometer_bottom, origin xyz=0 -0.14 0 rpy=1.5708 0 0
- added joint left_fr3_link2_accelerometer_top_joint: type fixed, parent left_fr3_link2, child left_fr3_link2_accelerometer_top, origin xyz=0 -0.13 0 rpy=-1.5708 0 0
- added joint left_fr3_link3_accelerometer_bottom_joint: type fixed, parent left_fr3_link3, child left_fr3_link3_accelerometer_bottom, origin xyz=0.0825 0.04 0 rpy=1.5708 0 0
- added joint left_fr3_link3_accelerometer_top_joint: type fixed, parent left_fr3_link3, child left_fr3_link3_accelerometer_top, origin xyz=0.0825 0.05 0 rpy=-1.5708 0 0
- added joint left_fr3_link4_accelerometer_bottom_joint: type fixed, parent left_fr3_link4, child left_fr3_link4_accelerometer_bottom, origin xyz=-0.0825 0.06 0 rpy=-1.5708 0 0
- added joint left_fr3_link4_accelerometer_top_joint: type fixed, parent left_fr3_link4, child left_fr3_link4_accelerometer_top, origin xyz=-0.0825 0.05 0 rpy=1.5708 0 0
- added joint left_fr3_link5_accelerometer_bottom_joint: type fixed, parent left_fr3_link5, child left_fr3_link5_accelerometer_bottom, origin xyz=0 0.1 0 rpy=1.5708 0 0
- added joint left_fr3_link5_accelerometer_top_joint: type fixed, parent left_fr3_link5, child left_fr3_link5_accelerometer_top, origin xyz=0 0.11 0 rpy=-1.5708 0 0
- added joint right_fr3_finger_joint1: type prismatic, parent right_fr3_hand, child right_fr3_leftfinger, origin xyz=0 0 0.0584 rpy=0 0 0, axis 0 1 0, limit lower=0.0 upper=0.04 effort=100 velocity=0.2
- added joint right_fr3_finger_joint2: type prismatic, parent right_fr3_hand, child right_fr3_rightfinger, origin xyz=0 0 0.0584 rpy=0 0 3.141592653589793, axis 0 1 0, limit lower=0.0 upper=0.04 effort=100 velocity=0.2, mimic joint=right_fr3_finger_joint1
- added joint right_fr3_hand_joint: type fixed, parent right_fr3_link8, child right_fr3_hand, origin xyz=0 0 0 rpy=0 0 -0.7853981633974483
- added joint right_fr3_hand_tcp_joint: type fixed, parent right_fr3_hand, child right_fr3_hand_tcp, origin xyz=0 0 0.1034 rpy=0 0 0
- added joint right_fr3_joint1: type revolute, parent right_fr3_link0, child right_fr3_link1, origin xyz=0 0 0.333 rpy=0 0 0, axis 0 0 1, limit lower=-2.9007400166666666 upper=2.9007400166666666 effort=87.0 velocity=2.62
- added joint right_fr3_joint2: type revolute, parent right_fr3_link1, child right_fr3_link2, origin xyz=0 0 0 rpy=-1.570796326794897 0 0, axis 0 0 1, limit lower=-1.8360900166666667 upper=1.8360900166666667 effort=87.0 velocity=2.62
- added joint right_fr3_joint3: type revolute, parent right_fr3_link2, child right_fr3_link3, origin xyz=0 -0.316 0 rpy=1.570796326794897 0 0, axis 0 0 1, limit lower=-2.9007400166666666 upper=2.9007400166666666 effort=87.0 velocity=2.62
- added joint right_fr3_joint4: type revolute, parent right_fr3_link3, child right_fr3_link4, origin xyz=0.0825 0 0 rpy=1.570796326794897 0 0, axis 0 0 1, limit lower=-3.077020016666667 upper=-0.11693708333333333 effort=87.0 velocity=2.62
- added joint right_fr3_joint5: type revolute, parent right_fr3_link4, child right_fr3_link5, origin xyz=-0.0825 0.384 0 rpy=-1.570796326794897 0 0, axis 0 0 1, limit lower=-2.87630335 upper=2.87630335 effort=12.0 velocity=5.26
- added joint right_fr3_joint6: type revolute, parent right_fr3_link5, child right_fr3_link6, origin xyz=0 0 0 rpy=1.570796326794897 0 0, axis 0 0 1, limit lower=0.43982265 upper=4.62163335 effort=12.0 velocity=4.18
- added joint right_fr3_joint7: type revolute, parent right_fr3_link6, child right_fr3_link7, origin xyz=0.088 0 0 rpy=1.570796326794897 0 0, axis 0 0 1, limit lower=-3.05083335 upper=3.05083335 effort=12.0 velocity=5.26
- added joint right_fr3_joint8: type fixed, parent right_fr3_link7, child right_fr3_link8, origin xyz=0 0 0.107 rpy=0 0 0
- added joint right_fr3_link0_accelerometer_bottom_joint: type fixed, parent right_fr3_link0, child right_fr3_link0_accelerometer_bottom, origin xyz=0 0 0.06 rpy=0 0 0
- added joint right_fr3_link0_accelerometer_top_joint: type fixed, parent right_fr3_link0, child right_fr3_link0_accelerometer_top, origin xyz=0 0 0.05 rpy=3.14159 0 0
- added joint right_fr3_link1_accelerometer_bottom_joint: type fixed, parent right_fr3_link1, child right_fr3_link1_accelerometer_bottom, origin xyz=0 -0.09 0.0 rpy=-1.5708 0 0
- added joint right_fr3_link1_accelerometer_top_joint: type fixed, parent right_fr3_link1, child right_fr3_link1_accelerometer_top, origin xyz=0 -0.1 0.0 rpy=1.5708 0 0
- added joint right_fr3_link2_accelerometer_bottom_joint: type fixed, parent right_fr3_link2, child right_fr3_link2_accelerometer_bottom, origin xyz=0 -0.14 0 rpy=1.5708 0 0
- added joint right_fr3_link2_accelerometer_top_joint: type fixed, parent right_fr3_link2, child right_fr3_link2_accelerometer_top, origin xyz=0 -0.13 0 rpy=-1.5708 0 0
- added joint right_fr3_link3_accelerometer_bottom_joint: type fixed, parent right_fr3_link3, child right_fr3_link3_accelerometer_bottom, origin xyz=0.0825 0.04 0 rpy=1.5708 0 0
- added joint right_fr3_link3_accelerometer_top_joint: type fixed, parent right_fr3_link3, child right_fr3_link3_accelerometer_top, origin xyz=0.0825 0.05 0 rpy=-1.5708 0 0
- added joint right_fr3_link4_accelerometer_bottom_joint: type fixed, parent right_fr3_link4, child right_fr3_link4_accelerometer_bottom, origin xyz=-0.0825 0.06 0 rpy=-1.5708 0 0
- added joint right_fr3_link4_accelerometer_top_joint: type fixed, parent right_fr3_link4, child right_fr3_link4_accelerometer_top, origin xyz=-0.0825 0.05 0 rpy=1.5708 0 0
- added joint right_fr3_link5_accelerometer_bottom_joint: type fixed, parent right_fr3_link5, child right_fr3_link5_accelerometer_bottom, origin xyz=0 0.1 0 rpy=1.5708 0 0
- added joint right_fr3_link5_accelerometer_top_joint: type fixed, parent right_fr3_link5, child right_fr3_link5_accelerometer_top, origin xyz=0 0.11 0 rpy=-1.5708 0 0
- added joint right_fr3_right_base_joint: type fixed, parent right_base, child right_fr3_link0, origin xyz=0 0 0 rpy=0 0 0
