Commit message: heartbeat for collision_node and check for running

File: franka_selfcollision/test/fr3_duo.urdf (robot description, URDF)
Before this commit: robot fr3_duo, 54 links, 53 joints
Links:
- removed link left_fr3_hand
- removed link left_fr3_hand_tcp
- removed link left_fr3_leftfinger
- removed link left_fr3_rightfinger
- removed link right_fr3_hand
- removed link right_fr3_hand_tcp
- removed link right_fr3_leftfinger
- removed link right_fr3_rightfinger
Joints:
- removed joint left_fr3_finger_joint1
- removed joint left_fr3_finger_joint2
- removed joint left_fr3_hand_joint
- removed joint left_fr3_hand_tcp_joint
- removed joint right_fr3_finger_joint1
- removed joint right_fr3_finger_joint2
- removed joint right_fr3_hand_joint
- removed joint right_fr3_hand_tcp_joint
