Commit message: fix: franka_description 2.4.0

File: franka_hardware/test/fr3.urdf (robot description, URDF)
Before this commit: robot fr3, 10 links, 9 joints
Links:
- link fr3_link0: geometry collision mesh filename=package://franka_description/meshes/robots/fr3/collision/li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; visual mesh filename=package://franka_description/meshes/robots/fr3/visual/link0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
- link fr3_link1: geometry collision mesh filename=package://franka_description/meshes/robots/fr3/collision/li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; visual mesh filename=package://franka_description/meshes/robots/fr3/visual/link1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
- link fr3_link2: geometry collision mesh filename=package://franka_description/meshes/robots/fr3/collision/li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; visual mesh filename=package://franka_description/meshes/robots/fr3/visual/link2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
- link fr3_link3: geometry collision mesh filename=package://franka_description/meshes/robots/fr3/collision/li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; visual mesh filename=package://franka_description/meshes/robots/fr3/visual/link3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
- link fr3_link4: geometry collision mesh filename=package://franka_description/meshes/robots/fr3/collision/li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; visual mesh filename=package://franka_description/meshes/robots/fr3/visual/link4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
- link fr3_link5: geometry collision mesh filename=package://franka_description/meshes/robots/fr3/collision/li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; visual mesh filename=package://franka_description/meshes/robots/fr3/visual/link5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
- link fr3_link6: geometry collision mesh filename=package://franka_description/meshes/robots/fr3/collision/li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; visual mesh filename=package://franka_description/meshes/robots/fr3/visual/link6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
- link fr3_link7: geometry collision mesh filename=package://franka_description/meshes/robots/fr3/collision/li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; visual mesh filename=package://franka_description/meshes/robots/fr3/visual/link7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

File: franka_hardware/test/fr3_unsupported_version.urdf (robot description, URDF)
Before this commit: robot fr3, 10 links, 9 joints
Links:
- link fr3_link0: geometry collision mesh filename=package://franka_description/meshes/robots/fr3/collision/li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; visual mesh filename=package://franka_description/meshes/robots/fr3/visual/link0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
- link fr3_link1: geometry collision mesh filename=package://franka_description/meshes/robots/fr3/collision/li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; visual mesh filename=package://franka_description/meshes/robots/fr3/visual/link1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
- link fr3_link2: geometry collision mesh filename=package://franka_description/meshes/robots/fr3/collision/li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; visual mesh filename=package://franka_description/meshes/robots/fr3/visual/link2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
- link fr3_link3: geometry collision mesh filename=package://franka_description/meshes/robots/fr3/collision/li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; visual mesh filename=package://franka_description/meshes/robots/fr3/visual/link3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
- link fr3_link4: geometry collision mesh filename=package://franka_description/meshes/robots/fr3/collision/li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; visual mesh filename=package://franka_description/meshes/robots/fr3/visual/link4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
- link fr3_link5: geometry collision mesh filename=package://franka_description/meshes/robots/fr3/collision/li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; visual mesh filename=package://franka_description/meshes/robots/fr3/visual/link5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
- link fr3_link6: geometry collision mesh filename=package://franka_description/meshes/robots/fr3/collision/li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; visual mesh filename=package://franka_description/meshes/robots/fr3/visual/link6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
- link fr3_link7: geometry collision mesh filename=package://franka_description/meshes/robots/fr3/collision/li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; visual mesh filename=package://franka_description/meshes/robots/fr3/visual/link7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

File: franka_selfcollision/test/fr3_duo.urdf (robot description, URDF)
Before this commit: robot fr3_duo, 46 links, 45 joints
Links:
- link left_fr3_link0: geometry collision mesh filename=package://franka_description/meshes/robots/fr3/collision/li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; visual mesh filename=package://franka_description/meshes/robots/fr3/visual/link0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
- link left_fr3_link1: geometry collision mesh filename=package://franka_description/meshes/robots/fr3/collision/li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; visual mesh filename=package://franka_description/meshes/robots/fr3/visual/link1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
- link left_fr3_link2: geometry collision mesh filename=package://franka_description/meshes/robots/fr3/collision/li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; visual mesh filename=package://franka_description/meshes/robots/fr3/visual/link2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
- link left_fr3_link3: geometry collision mesh filename=package://franka_description/meshes/robots/fr3/collision/li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; visual mesh filename=package://franka_description/meshes/robots/fr3/visual/link3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
- link left_fr3_link4: geometry collision mesh filename=package://franka_description/meshes/robots/fr3/collision/li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; visual mesh filename=package://franka_description/meshes/robots/fr3/visual/link4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
- link left_fr3_link5: geometry collision mesh filename=package://franka_description/meshes/robots/fr3/collision/li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; visual mesh filename=package://franka_description/meshes/robots/fr3/visual/link5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
- link left_fr3_link6: geometry collision mesh filename=package://franka_description/meshes/robots/fr3/collision/li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; visual mesh filename=package://franka_description/meshes/robots/fr3/visual/link6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
- link left_fr3_link7: geometry collision mesh filename=package://franka_description/meshes/robots/fr3/collision/li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; visual mesh filename=package://franka_description/meshes/robots/fr3/visual/link7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
- link right_fr3_link0: geometry collision mesh filename=package://franka_description/meshes/robots/fr3/collision/li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; visual mesh filename=package://franka_description/meshes/robots/fr3/visual/link0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
- link right_fr3_link1: geometry collision mesh filename=package://franka_description/meshes/robots/fr3/collision/li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; visual mesh filename=package://franka_description/meshes/robots/fr3/visual/link1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
- link right_fr3_link2: geometry collision mesh filename=package://franka_description/meshes/robots/fr3/collision/li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; visual mesh filename=package://franka_description/meshes/robots/fr3/visual/link2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
- link right_fr3_link3: geometry collision mesh filename=package://franka_description/meshes/robots/fr3/collision/li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; visual mesh filename=package://franka_description/meshes/robots/fr3/visual/link3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
- link right_fr3_link4: geometry collision mesh filename=package://franka_description/meshes/robots/fr3/collision/li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; visual mesh filename=package://franka_description/meshes/robots/fr3/visual/link4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
- link right_fr3_link5: geometry collision mesh filename=package://franka_description/meshes/robots/fr3/collision/li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; visual mesh filename=package://franka_description/meshes/robots/fr3/visual/link5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
- link right_fr3_link6: geometry collision mesh filename=package://franka_description/meshes/robots/fr3/collision/li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; visual mesh filename=package://franka_description/meshes/robots/fr3/visual/link6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
- link right_fr3_link7: geometry collision mesh filename=package://franka_description/meshes/robots/fr3/collision/li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; visual mesh filename=package://franka_description/meshes/robots/fr3/visual/link7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
