Commit message: feat: Add Gazebo URDF entry points, sensor plugins, and example worlds

File: franka_gazebo_bringup/urdf/sensors.xacro (robot description, xacro)
@@ -24,3 +24,97 @@
         <xacro:franka_gazebo_imu link_target="${prefix}_link5_accelerometer_${imu_side}" gz_topic="/${prefix}/imu/link5/${imu_side}"/>
     </xacro:macro>
+    <xacro:macro name="franka_gazebo_camera" params="link_reference sensor_name gz_topic
+                 rate:=30 hfov:=1.047 width:=640 height:=480 format:=R8G8B8
+                 clip_near:=0.1 clip_far:=100.0 visualize:=true">
+        <gazebo reference="${link_reference}">
+            <sensor name="${sensor_name}" type="camera">
+                <pose>0 0 0 0 0 0</pose>
+                <topic>${gz_topic}</topic>
+                <update_rate>${rate}</update_rate>
+                <camera>
+                    <horizontal_fov>${hfov}</horizontal_fov>
+                    <image>
+                        <width>${width}</width>
+                        <height>${height}</height>
+                        <format>${format}</format>
+                    </image>
+                    <clip>
+                        <near>${clip_near}</near>
+                        <far>${clip_far}</far>
+                    </clip>
+                </camera>
+                <always_on>true</always_on>
+                <visualize>${visualize}</visualize>
+            </sensor>
+        </gazebo>
+    </xacro:macro>
+    <!-- ================= LIDAR MACRO ================= -->
+    <xacro:macro name="franka_gazebo_lidar" params="link_reference sensor_name ros_topic
+                 update_rate:=50.0 min_angle:='${radians(-45)}' max_angle:='${radians(225)}'
+                 min_range:=0.05 max_range:=10.0 max_beams:=500
+                 gaussian_noise:=0.006">
+        <plugin
+          filename="gz-sim-sensors-system"
+          name="gz::sim::systems::Sensors">
+          <render_engine>ogre2</render_engine>
+        </plugin>
+        <gazebo reference="${link_reference}">
+            <material value="Gazebo/Yellow" />
+            <sensor name="${sensor_name}" type="gpu_lidar">
+                <topic>${ros_topic}</topic>
+                <update_rate>${update_rate}</update_rate>
+                <gz_frame_id>${link_reference}</gz_frame_id>
+                <lidar>
+                    <scan>
+                        <horizontal>
+                            <samples>${max_beams}</samples>
+                            <resolution>1</resolution>
+                            <min_angle>${min_angle}</min_angle>
+                            <max_angle>${max_angle}</max_angle>
+                        </horizontal>
+                        <vertical>
+                            <samples>16</samples>
+                            <resolution>1</resolution>
+                            <min_angle>-0.261799</min_angle>
+                            <max_angle>0.261799</max_angle>
+                        </vertical>
+                    </scan>
+                    <range>
+                        <min>${min_range}</min>
+                        <max>${max_range}</max>
+                        <resolution>0.01</resolution>
+                    </range>
+                    <noise>
+                        <type>gaussian</type>
+                        <mean>0.0</mean>
+                        <stddev>${gaussian_noise}</stddev>
+                    </noise>
+                </lidar>
+                <visualize>true</visualize>
+            </sensor>
+        </gazebo>
+    </xacro:macro>
+    <!-- ================= BODY IMU MACRO ================= -->
+    <xacro:macro name="franka_gazebo_body_imu" params="link_reference gz_topic rate:=100
+                 gyro_stddev:=0.009 accel_stddev:=0.021">
+        <gazebo reference="${link_reference}">
+            <sensor name="imu_sensor" type="imu">
+                <topic>${gz_topic}</topic>
+                <update_rate>${rate}</update_rate>
+                <always_on>true</always_on>
+                <imu>
+                    <angular_velocity>
+                        <x><noise type="gaussian"><mean>0</mean><stddev>${gyro_stddev}</stddev></noise></x>
+                        <y><noise type="gaussian"><mean>0</mean><stddev>${gyro_stddev}</stddev></noise></y>
+                        <z><noise type="gaussian"><mean>0</mean><stddev>${gyro_stddev}</stddev></noise></z>
+                    </angular_velocity>
+                    <linear_acceleration>
+                        <x><noise type="gaussian"><mean>0</mean><stddev>${accel_stddev}</stddev></noise></x>
+                        <y><noise type="gaussian"><mean>0</mean><stddev>${accel_stddev}</stddev></noise></y>
+                        <z><noise type="gaussian"><mean>0</mean><stddev>${accel_stddev}</stddev></noise></z>
+                    </linear_acceleration>
+                </imu>
+            </sensor>
+        </gazebo>
+    </xacro:macro>
 </robot>
