Commit message: Refactors Gazebo gravity overrides for robots
Extracts gravity override configurations for Franka arms and mobile bases into a reusable `gravity_overrides.xacro` file. This centralizes the logic to disable gravity on specific links and apply implicit spring damping where necessary.

Updates launch files to utilize a consolidated `franka_arm.gazebo.xacro` for arm descriptions, which now includes the arm-specific gravity overrides.

These changes prevent robot arms from collapsing in Gazebo simulations when using example controllers that do not implement gravity compensation. The refactoring improves maintainability and reduces duplication across various robot configurations.

File: franka_gazebo_bringup/urdf/franka_arm.gazebo.xacro (robot description, xacro)
@@ -6,7 +6,11 @@
     <!-- Include gazebo macros -->
     <xacro:include filename="$(find franka_gazebo_bringup)/urdf/sensors.xacro"/>
+    <xacro:include filename="$(find franka_gazebo_bringup)/urdf/gravity_overrides.xacro"/>
     <!-- Arm IMUs -->
     <!-- arm prefix is inherited from the franka_description xacro -->
     <xacro:franka_gazebo_arm_imus arm_prefix="$(arg arm_prefix)" robot_type="$(arg robot_type)" imu_side="top"/>
     <xacro:franka_gazebo_arm_imus arm_prefix="$(arg arm_prefix)" robot_type="$(arg robot_type)" imu_side="bottom"/>
+    <!-- Disable gravity on arm links: the example controllers do not
+         implement gravity compensation, so the arms would collapse. -->
+    <xacro:disable_arm_gravity prefix="$(arg arm_prefix)" robot_type="$(arg robot_type)"/>
 </robot>

File: franka_gazebo_bringup/urdf/mobile_fr3_duo_v0_2.gazebo.urdf.xacro (robot description, xacro)
@@ -16,4 +16,5 @@
   <!-- ================================================================ -->
   <xacro:include filename="$(find franka_description)/robots/mobile_fr3_duo_v0_2/mobile_fr3_duo_v0_2.xacro"/>
+  <xacro:include filename="$(find franka_gazebo_bringup)/urdf/gravity_overrides.xacro"/>
   <!-- ================================================================ -->
   <!-- Arguments                                                        -->
@@ -69,35 +70,6 @@
   <!-- Gravity overrides                                                -->
   <!-- ================================================================ -->
-  <!-- Disable gravity on arm links: the example controllers do not
-       implement gravity compensation, so the arms would collapse. -->
-  <xacro:macro name="disable_arm_gravity" params="prefix robot_type">
-    <gazebo reference="${prefix}${robot_type}_link0"><gravity>false</gravity></gazebo>
-    <gazebo reference="${prefix}${robot_type}_link1"><gravity>false</gravity></gazebo>
-    <gazebo reference="${prefix}${robot_type}_link2"><gravity>false</gravity></gazebo>
-    <gazebo reference="${prefix}${robot_type}_link3"><gravity>false</gravity></gazebo>
-    <gazebo reference="${prefix}${robot_type}_link4"><gravity>false</gravity></gazebo>
-    <gazebo reference="${prefix}${robot_type}_link5"><gravity>false</gravity></gazebo>
-    <gazebo reference="${prefix}${robot_type}_link6"><gravity>false</gravity></gazebo>
-    <gazebo reference="${prefix}${robot_type}_link7"><gravity>false</gravity></gazebo>
-    <gazebo reference="${prefix}${robot_type}_link8"><gravity>false</gravity></gazebo>
-    <gazebo reference="${prefix}${robot_type}_flange"><gravity>false</gravity></gazebo>
-    <gazebo reference="${prefix}${robot_type}_hand"><gravity>false</gravity></gazebo>
-    <gazebo reference="${prefix}${robot_type}_leftfinger"><gravity>false</gravity></gazebo>
-    <gazebo reference="${prefix}${robot_type}_rightfinger"><gravity>false</gravity></gazebo>
-  </xacro:macro>
   <xacro:disable_arm_gravity prefix="left_" robot_type="${robot_types_list[1]}"/>
   <xacro:disable_arm_gravity prefix="right_" robot_type="${robot_types_list[2]}"/>
-  <!-- Disable gravity on spine links so the lift does not sag. -->
-  <gazebo reference="franka_spine"><gravity>false</gravity></gazebo>
-  <gazebo reference="franka_spine_support"><gravity>false</gravity></gazebo>
-  <gazebo reference="mount_link"><gravity>false</gravity></gazebo>
-  <gazebo reference="head_link"><gravity>false</gravity></gazebo>
-  <!-- Hold the spine lift joint against reaction forces.
-       The stiffness resists displacement, the damping prevents oscillation.
-       A commanded position change can still overcome these values. -->
-  <gazebo reference="franka_spine_vertical_joint">
-    <implicitSpringDamper>true</implicitSpringDamper>
-    <springStiffness>5000</springStiffness>
-    <springDamping>500</springDamping>
-  </gazebo>
+  <xacro:disable_mobile_base_gravity/>
 </robot>

File: franka_gazebo_bringup/urdf/mobile_fr3_duo_v0_2_with_sensors.gazebo.urdf.xacro (robot description, xacro)
@@ -20,4 +20,5 @@
   <xacro:include filename="$(find franka_mobile_sensors)/robots/mobile_fr3_duo_v0_2_with_sensors.xacro"/>
   <xacro:include filename="$(find franka_gazebo_bringup)/urdf/sensors.xacro" />
+  <xacro:include filename="$(find franka_gazebo_bringup)/urdf/gravity_overrides.xacro"/>
   <!-- ================================================================ -->
   <!-- Arguments                                                        -->
@@ -96,35 +97,6 @@
   <!-- Gravity overrides                                                -->
   <!-- ================================================================ -->
-  <!-- Disable gravity on arm links: the example controllers do not
-       implement gravity compensation, so the arms would collapse. -->
-  <xacro:macro name="disable_arm_gravity" params="prefix robot_type">
-    <gazebo reference="${prefix}${robot_type}_link0"><gravity>false</gravity></gazebo>
-    <gazebo reference="${prefix}${robot_type}_link1"><gravity>false</gravity></gazebo>
-    <gazebo reference="${prefix}${robot_type}_link2"><gravity>false</gravity></gazebo>
-    <gazebo reference="${prefix}${robot_type}_link3"><gravity>false</gravity></gazebo>
-    <gazebo reference="${prefix}${robot_type}_link4"><gravity>false</gravity></gazebo>
-    <gazebo reference="${prefix}${robot_type}_link5"><gravity>false</gravity></gazebo>
-    <gazebo reference="${prefix}${robot_type}_link6"><gravity>false</gravity></gazebo>
-    <gazebo reference="${prefix}${robot_type}_link7"><gravity>false</gravity></gazebo>
-    <gazebo reference="${prefix}${robot_type}_link8"><gravity>false</gravity></gazebo>
-    <gazebo reference="${prefix}${robot_type}_flange"><gravity>false</gravity></gazebo>
-    <gazebo reference="${prefix}${robot_type}_hand"><gravity>false</gravity></gazebo>
-    <gazebo reference="${prefix}${robot_type}_leftfinger"><gravity>false</gravity></gazebo>
-    <gazebo reference="${prefix}${robot_type}_rightfinger"><gravity>false</gravity></gazebo>
-  </xacro:macro>
   <xacro:disable_arm_gravity prefix="left_" robot_type="${robot_types_list[1]}"/>
   <xacro:disable_arm_gravity prefix="right_" robot_type="${robot_types_list[2]}"/>
-  <!-- Disable gravity on spine links so the lift does not sag. -->
-  <gazebo reference="franka_spine"><gravity>false</gravity></gazebo>
-  <gazebo reference="franka_spine_support"><gravity>false</gravity></gazebo>
-  <gazebo reference="mount_link"><gravity>false</gravity></gazebo>
-  <gazebo reference="head_link"><gravity>false</gravity></gazebo>
-  <!-- Hold the spine lift joint against reaction forces.
-       The stiffness resists displacement, the damping prevents oscillation.
-       A commanded position change can still overcome these values. -->
-  <gazebo reference="franka_spine_vertical_joint">
-    <implicitSpringDamper>true</implicitSpringDamper>
-    <springStiffness>5000</springStiffness>
-    <springDamping>500</springDamping>
-  </gazebo>
+  <xacro:disable_mobile_base_gravity/>
 </robot>
